File: KiCad/ESP32_PortableDA/ESP32_BTDA.kicad_sch (KiCad schematic)
At the start: 47 parts, among them J1 USB_C_Receptacle_USB2.0, J2 AudioJack3_Ground, J3 JST_BattConn, Q1 Q_PMOS, U1 PCM5100APWR, U2 TPA6133A2RTJR, U3 BQ25308RTER, U4 TLV74033PDBVR-A, U5 TLV74033PDBVR-D

Commit message: Fixed problems with BC and DAC schematics
Parts:
- U1: footprint ECE402FinalProj:PCM5100APWR -> Package_SO:TSSOP-20_4.4x6.5mm_P0.65mm; Mfg (none) -> Texas Instruments; Part No. (none) -> PCM5100APWR; Supplier 1 (none) -> https://www.digikey.com/en/products/detail/texas-instrument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; Supplier 2 (none) -> https://www.lcsc.com/search?q=PCM5100APWR&s_z=n_PCM5100APWR
Other:
- note removed: "02/06/2026"
- note removed: "ESP32 Portable Bluetooth DAC/AMP"
- company: (none) -> ECE402
- title: (none) -> ESP32 Bluetooth DAC/AMP
Changed lines of the file:
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@@
 	(generator_version "9.0")
 	(paper "A")
+	(title_block
+		(title "ESP32 Bluetooth DAC/AMP")
+		(date "2026-02-19")
+		(rev "A")
+		(company "ECE402")
+	)
 	(rectangle
 		(start 164.592 53.848)
@@
 		)
 	)
-	(text "02/06/2026"
-		(exclude_from_sim no)
-		(at 188.468 199.898 0)
-		(effects
-			(font
-				(size 1.27 1.27)
-			)
-			(justify left bottom)
-		)
-	)
 	(text "Add value for:\nQ1\nD1,2\nR7, 8\nL1"
 		(exclude_from_sim no)
@@
 		)
 	)
-	(text "ESP32 Portable Bluetooth DAC/AMP"
-		(exclude_from_sim no)
-		(at 168.148 196.85 0)
-		(effects
-			(font
-				(size 2 2)
-			)
-			(justify left bottom)
-		)
-	)
 	(text "Add footprint for:\nQ1\nD1,2"
 		(exclude_from_sim no)
@@
 	)
 	(symbol
-		(lib_id "ECE402FinalProj:PCM5100APWR")
-		(at 220.98 45.72 0)
-		(unit 1)
-		(exclude_from_sim no)
-		(in_bom yes)
-		(on_board yes)
-		(dnp no)
-		(fields_autoplaced yes)
-		(property "Reference" "U1"
-			(at 220.98 51.562 0)
-			(effects
-				(font
-					(size 1.524 1.524)
-				)
-			)
-		)
-		(property "Value" "PCM5100APWR"
-			(at 220.98 55.372 0)
-			(effects
-				(font
-					(size 1.524 1.524)
-				)
-			)
-		)
-		(property "Footprint" "ECE402FinalProj:PCM5100APWR"
-			(at 218.44 48.26 0)
-			(effects
-				(font
-					(size 1.27 1.27)
-					(italic yes)
-				)
-				(hide yes)
-			)
-		)
-		(property "Datasheet" "https://www.ti.com/lit/gpn/pcm5100a"
-			(at 218.44 48.26 0)
-			(effects
-				(font
-					(size 1.27 1.27)
-					(italic yes)
-				)
-				(hide yes)
-			)
-		)
-		(property "Description" ""
-			(at 220.98 45.72 0)
-			(effects
-				(font
-					(size 1.27 1.27)
-				)
-				(hide yes)
-			)
-		)
-		(pin "8"
-		)
-		(pin "10"
-		)
-		(pin "1"
-		)
-		(pin "14"
-		)
-		(pin "20"
-		)
-		(pin "12"
-		)
-		(pin "19"
-		)
-		(pin "15"
-		)
-		(pin "7"
-		)
-		(pin "4"
-		)
-		(pin "13"
-		)
-		(pin "11"
-		)
-		(pin "6"
-		)
-		(pin "2"
-		)
-		(pin "5"
-		)
-		(pin "16"
-		)
-		(pin "17"
-		)
-		(pin "9"
-		)
-		(pin "18"
-		)
-		(pin "3"
-		)
-		(instances
-			(project ""
-				(path "/b3b9d018-954a-4fab-ac7e-c234f13b80c6"
-					(reference "U1")
-					(unit 1)
-				)
-			)
-		)
-	)
-	(symbol
 		(lib_id "Device:C")
 		(at 52.07 91.44 0)
@@
 	)
 	(symbol
+		(lib_id "ECE402FinalProj:PCM5100APWR")
+		(at 208.28 19.05 0)
+		(unit 1)
+		(exclude_from_sim no)
+		(in_bom yes)
+		(on_board yes)
+		(dnp no)
+		(fields_autoplaced yes)
+		(property "Reference" "U1"
+			(at 220.98 13.97 0)
+			(effects
+				(font
+					(size 1.524 1.524)
+				)
+			)
+		)
+		(property "Value" "PCM5100APWR"
+			(at 220.98 16.51 0)
+			(effects
+				(font
+					(size 1.524 1.524)
+				)
+			)
+		)
+		(property "Footprint" "Package_SO:TSSOP-20_4.4x6.5mm_P0.65mm"
+			(at 268.224 40.64 0)
+			(effects
+				(font
+					(size 1.27 1.27)
+					(italic yes)
+				)
+				(hide yes)
+			)
+		)
+		(property "Datasheet" "https://www.ti.com/lit/gpn/pcm5100a"
+			(at 272.288 47.752 0)
+			(effects
+				(font
+					(size 1.27 1.27)
+					(italic yes)
+				)
+				(hide yes)
+			)
+		)
+		(property "Description" "IC DAC 16/24/32BIT 384K 20TSSOP"
+			(at 271.018 44.196 0)
+			(effects
+				(font
+					(size 1.27 1.27)
+				)
+				(hide yes)
+			)
+		)
+		(property "Mfg" "Texas Instruments"
+			(at 261.874 50.8 0)
+			(effects
+				(font
+					(size 1.27 1.27)
+				)
+				(hide yes)
+			)
+		)
+		(property "Part No." "PCM5100APWR"
+			(at 260.096 54.102 0)
+			(effects
+				(font
+					(size 1.27 1.27)
+				)
+				(hide yes)
+			)
+		)
+		(property "Supplier 1" "https://www.digikey.com/en/products/detail/texas-instruments/PCM5100APWR/4341332?gclsrc=aw.ds&gad_source=1&gad_campaignid=17338792030&gbraid=0AAAAADrbLlikoHYVm1EAT8Ro0lFRq30vw&gclid=CjwKCAiAv5bMBhAIEiwAqP9GuJ40P9n3nzht8Krs9izPPDkGNq60HQeCsuY7D_maf0OzrZdjZgSlNBoC1acQAvD_BwE"
+			(at 406.146 57.404 0)
+			(effects
+				(font
+					(size 1.27 1.27)
+				)
+				(hide yes)
+			)
+		)
+		(property "Supplier 2" "https://www.lcsc.com/search?q=PCM5100APWR&s_z=n_PCM5100APWR"
+			(at 287.274 60.706 0)
+			(effects
+				(font
+					(size 1.27 1.27)
+				)
+				(hide yes)
+			)
+		)
+		(pin "20"
+		)
+		(pin "16"
+		)
+		(pin "3"
+		)
+		(pin "7"
+		)
+		(pin "10"
+		)
+		(pin "17"
+		)
+		(pin "8"
+		)
+		(pin "11"
+		)
+		(pin "14"
+		)
+		(pin "13"
+		)
+		(pin "4"
+		)
+		(pin "9"
+		)
+		(pin "6"
+		)
+		(pin "12"
+		)
+		(pin "15"
+		)
+		(pin "18"
+		)
+		(pin "19"
+		)
+		(pin "2"
+		)
+		(pin "5"
+		)
+		(pin "1"
+		)
+		(instances
+			(project ""
+				(path "/b3b9d018-954a-4fab-ac7e-c234f13b80c6"
+					(reference "U1")
+					(unit 1)
+				)
+			)
+		)
+	)
+	(symbol
 		(lib_id "Device:C_Small")
 		(at 195.58 63.5 0)
@@
 					(size 1.27 1.27)
 				)
+				(hide yes)
 			)
 		)
@@
 	(symbol
 		(lib_id "ECE402FinalProj:BQ25308RTER")
-		(at 115.57 46.99 0)
+		(at 102.87 33.02 0)
 		(unit 1)
 		(exclude_from_sim no)
@@
 		(on_board yes)
 		(dnp no)
-		(fields_autoplaced yes)
 		(property "Reference" "U3"
-			(at 115.824 46.228 0)
+			(at 104.648 31.75 0)
 			(effects
 				(font
@@
 		)
 		(property "Value" "BQ25308RTER"
-			(at 115.824 48.768 0)
+			(at 125.222 64.008 0)
 			(effects
 				(font
@@
 		)
 		(property "Footprint" "WQFN16_RTE_TEX"
-			(at 95.25 35.56 0)
+			(at 147.828 55.626 0)
 			(effects
 				(font
@@
 		)
 		(property "Datasheet" "https://www.ti.com/lit/gpn/bq25308"
-			(at 95.25 35.56 0)
+			(at 157.988 58.674 0)
 			(effects
 				(font
@@
 		)
 		(property "Description" ""
-			(at 115.57 46.99 0)
+			(at 102.87 33.02 0)
 			(effects
 				(font

Commit message: Updated Schematics
Full schematic with net labels and all footprints on board, missing some 3D models
Parts:
- removed C1: C, Capacitor_SMD:C_0603_1608Metric, symbol Device:C
- removed D2: D_Vbus, symbol Device:D_Small
- removed J1: USB_C_Receptacle_USB2.0, symbol Connector:USB_C_Receptacle_USB2.0
- removed J2: AudioJack3_Ground, symbol Connector_Audio:AudioJack3_Ground
- removed Q1: Q_PMOS, symbol Device:Q_PMOS
- removed R1, R8: R, Resistor_SMD:R_0603_1608Metric, symbol Device:R
- removed R2: R, Resistor_SMD:R_0402_1005Metric, symbol Device:R_Small
- removed U4: TLV74033PDBVR-A, DBV0005A-IPC_A, symbol ECE402FinalProj:TLV74033PDBVR
- removed U5: TLV74033PDBVR-D, DBV0005A-IPC_A, symbol ECE402FinalProj:TLV74033PDBVR
- added C1: 4p, Capacitor_SMD:C_0402_1005Metric, symbol Device:C_Small
- added C24, C26, C29: 1u, Capacitor_SMD:C_0603_1608Metric, symbol Device:C_Small
- added C25: 0.1n, Capacitor_SMD:C_0402_1005Metric, symbol Device:C_Small
- added C27, C30, C32, C33: 0u1, Capacitor_SMD:C_0402_1005Metric, symbol Device:C_Small
- added C28: 10u, Capacitor_SMD:C_0805_2012Metric, symbol Device:C_Small
- added C31: C, Capacitor_SMD:C_0603_1608Metric, symbol Device:C_Small
- added C34: 10n, Capacitor_SMD:C_0402_1005Metric, symbol Device:C_Small
- added C35: 3n3, Capacitor_SMD:C_0402_1005Metric, symbol Device:C_Small
- added C36, C37: C, Capacitor_SMD:C_0402_1005Metric, symbol Device:C_Small
- added C38, C39: 47n, Capacitor_SMD:C_0402_1005Metric, symbol Device:C_Small
- added C40, C41, C42, C43: 1u, Capacitor_SMD:C_0603_1608Metric, symbol Device:C
- added D2: ESD5Zxx, Diode_SMD:D_SOD-523, symbol Diode:ESD5Zxx
- added J1: ASJ-200-B-HT, ASJ-200-B-HT_ADM, symbol ECE402FinalProj:ASJ-200-B-HT
- added J2: USB_C_Receptacle_PowerOnly_6P, Connector_USB:USB_C_Receptacle_GCT_USB4125-xx-x_6P_TopMnt_Horizontal, symbol Connector:USB_C_Receptacle_PowerOnly_6P
- added J4: uart_conn, Connector_PinHeader_2.54mm:PinHeader_1x03_P2.54mm_Vertical, symbol Connector:Conn_01x03_Pin
- added L2, L3: 2n, Inductor_SMD:L_0402_1005Metric, symbol Device:L
- added R13: 2k, Resistor_SMD:R_0402_1005Metric, symbol Device:R_Small
- added R14: 10k, Resistor_SMD:R_0402_1005Metric, symbol Device:R_Small
- added R15: 20k, Resistor_SMD:R_0402_1005Metric, symbol Device:R_Small
- added R16: R, Resistor_SMD:R_0402_1005Metric, symbol Device:R_Small
- added R17, R18, R19, R20, R21, R22, R23, R24, R8: 0, Resistor_SMD:R_0402_1005Metric, symbol Device:R_Small
- added R25: 2k2, Resistor_SMD:R_0402_1005Metric, symbol Device:R_Small
- added S1: On switch, ECE402FinalProj:SW_SLW-129956-4A-RA-N-D, symbol ECE402FinalProj:SLW-129956-4A-RA-N-D
- added U4, U5: NCP177, Package_DFN_QFN:OnSemi_XDFN4-1EP_1.0x1.0mm_EP0.52x0.52mm, symbol ECE402FinalProj:NCP177BMX330TCG
- added U6: ESP32_D0WD_V3, Package_DFN_QFN:QFN-48-1EP_5x5mm_P0.35mm_EP3.7x3.7mm_ThermalVias, symbol ECE402FinalProj:ESP32
- added U8: BY25Q32ESSIG(R), Package_SO:SOP-8_3.76x4.96mm_P1.27mm, symbol ECE402FinalProj:BY25Q32ESSIG(R)
- added U9: AN043, ECE402FinalProj:AN043_2.4GHz_PCB_Antenna, symbol ECE402FinalProj:AN043
- added X1: ECS-400, Crystal:Crystal_SMD_2016-4Pin_2.0x1.6mm, symbol Device:Crystal_GND24_Small
- C11, C19, C22, C23, C7, C8, C9: footprint Capacitor_SMD:C_0402_1005Metric -> Capacitor_SMD:C_0805_2012Metric
- C12, C15, C16, C20: footprint Capacitor_SMD:C_0402_1005Metric -> Capacitor_SMD:C_0603_1608Metric
- C13, C14, C17, C21: footprint (none) -> Capacitor_SMD:C_0805_2012Metric
- C2: value C -> 5p
- C3: value 10u -> 1u
- C6: value 22u -> 1u; footprint Capacitor_SMD:C_0603_1608Metric -> Capacitor_SMD:C_0805_2012Metric
- D1: footprint (none) -> LED_SMD:LED_0603_1608Metric
- L1: value L -> 1u; footprint (none) -> Inductor_SMD:L_0805_2012Metric
- R5: value 1k0 -> 1k
- R6: value R -> 10k; now fitted
- R7: value R -> 13k
Connections:
- net GND: now also C2.2, U2.13 (GND), U2.19 (GND), C1.2, C24.2, C25.2, C26.2, C27.2, C28.2, C29.2, C30.2, C31.2, C32.2, C33.2, C34.2, C36.2, C37.2, C40.2, C41.2, C43.2, D2.2 (A), J1.1, J2.A12 (GND), J2.B12 (GND), J4.3 (Pin_3), R13.2, R17.1, R18.1, R19.1, R8.2, S1.3, U4.2 (GND), U5.2 (GND), U6.22 (GPIO2), U6.49 (GND), U8.4 (VSS), U9.1 (GND), X1.2 (G), X1.4 (G); no longer U1.10 (DEMP), U1.11 (FLT), U1.16 (FMT)
- net VAA: now also U2.12 (VDD), U2.20 (VDD), C25.1, C26.1, C27.1, C28.1, C29.1, C30.1, C40.1, C41.1, L2.1, R14.1, R25.1, S1.1, U4.1 (OUT), U6.1 (VDDA), U6.43 (VDDA), U6.46 (VDDA)
- net VDD: now also C32.1, C33.1, U5.1 (OUT), U6.19 (VDD3P3_RTC), U6.37 (VDD3P3_CPU)
- net bck: now also U6.35 (GPIO18)
- net din: now also U6.36 (GPIO23)
- net lrck: now also U6.38 (GPIO19)
- net ldoo: now reaches C12.1, C13.1, U1.18 (LDOO)
- net +BATT: now reaches C4.1
- net +BATT: now also C11.1, C5.1, J3.1 (Pin_1), L1.2, U3.10 (BAT), U4.4 (IN), U5.4 (IN)
- net pmid: now reaches C9.1, U3.16 (PMID)
- net btst: now reaches C10.1, U3.15 (BTST)
- net sw: now reaches C10.2, L1.1, U3.13 (SW), U3.14 (SW)
- net stat: now reaches R5.1, U3.3 (STAT)
- net dstat: now reaches D1.1 (K), R5.2
- net cc1: now reaches R4.1
- net cc1: now also J2.A5 (CC1)
- net cc2: now reaches R3.1
- net cc2: now also J2.B5 (CC2)
- net veng: now reaches C19.1, U1.5 (VNEG)
- net amp_lin: now reaches U2.1 (LEFTINM)
- net amp_lin: now also U2.2 (LEFTINP), C38.2
- net con_m: now reaches U2.11 (HPRIGHT)
- net con_m: now also J1.3
- net con_t: now reaches U2.14 (HPLEFT)
- net con_t: now also J1.2, J1.4
- net cpvss: now reaches U2.15 (CPVSS)
- net cpvss: now also U2.16 (CPVSS), C43.1
- net cpn: now reaches U2.17 (CPN)
- net cpn: now also C42.1
- net cpp: now reaches U2.18 (CPP)
- net cpp: now also C42.2
- net amp_rin: now reaches U2.4 (RIGHTINP)
- net amp_rin: now also U2.5 (RIGHTINM), C39.2
- net sd: now reaches U2.6 (*SD)
- net sd: now also U6.15 (GPIO26)
- net at U2.7 (TEST2): now also U2.8 (TEST1), R25.2
- net vset: now reaches R6.1, U3.9 (VSET)
- net outl: now reaches R11.1, U1.6 (OUTL)
- net ichg: now reaches R7.1, U3.4 (ICHG)
- net cap1: now reaches C18.1, U1.2 (CAPP)
- net cap1: now also C34.1, C35.1, R15.1, U6.48 (CAP1)
- net capm: now reaches C18.2, U1.4 (CAPM)
- net outr: now reaches R12.1, U1.7 (OUTR)
- net lna_in: now reaches C2.1
- net lna_in: now also L3.2, U6.2 (LNA_IN)
- net doutl renamed loutl
- net loutl: now also C38.1
- net doutr renamed loutr
- net loutr: now also C39.1
- net vbus renamed VBUS
- net VBUS: now also D2.1 (K), J2.A9 (VBUS), J2.B9 (VBUS)
- new net: R24.1, U6.33 (SD_DATA_1)
- new net: R14.2, U6.18 (MTDI)
- new net: R20.1, U6.28 (SD_DATA_2)
- new net: R22.1, U6.31 (SD_CLK)
- new net: R23.1, U6.32 (SD_DATA_0)
- new net: R21.1, U6.29 (SD_DATA_3)
- new net SCK/CLK: R22.2, U8.6 (SCLK)
- new net SCS/CMD: U6.30 (SD_CMD), U8.1 (/CS)
- new net SDI/SD1: R24.2, U8.5 (SI)
- new net SDO/SD0: R23.2, U8.2 (SO)
- new net SHD/SD2: R20.2, U8.7 (/HOLD)
- new net SWP/SD3: R21.2, U8.3 (/WP)
- new net VDD_SDIO: C24.1, R13.1, U6.26 (VDD_SDIO), U8.8 (VCC)
- new net ant_ino: C1.1, L3.1, U9.2 (FEED)
- new net boot: R8.1, U6.23 (GPIO0)
- new net cap2: C35.2, R15.2, U6.47 (CAP2)
- new net demp: R18.2, U1.10 (DEMP)
- new net en: S1.2, U4.3 (EN), U5.3 (EN), U6.9 (CHIP_PU)
- new net flt: R19.2, U1.11 (FLT)
- new net fmt: R17.2, U1.16 (FMT)
- new net uorxd: J4.2 (Pin_2), U6.40 (UORXD)
- new net uotxd: J4.1 (Pin_1), U6.41 (UOTXD)
- new net vdd3p3: C31.1, L2.2, U6.3 (VDD3P3), U6.4 (VDD3P3)
- new net x1: C37.1, R16.1, X1.1
- new net x3: C36.1, U6.44 (XTAL_N), X1.3
- new net xtalp: R16.2, U6.45 (XTAL_P)
- no-connect marks 6 -> 21
Other:
- note added: "Add footprint for:"
- note added: "Add value for: R16 C36, 37 SW1"
- note added: "Audio"
- note added: "CAPACITOR FOOTPRINT GUIDE: 0402 - C=<100nF 0603 - 100nF<C<2.2uF 0805 - C>=2.2uF size up if worried about derating/signal char."
- note added: "ESP/RF Circuitry"
- note added: "Est. after layout"
- note added: "Power Management/Delivery"
- note added: "With GPIO0/2 low part will enter serial loader otherwise it will boot from flash GPIO2 is ignored when 0 is hi"
- note removed: "0603 is for HP/analog and 0402 otherwise"
- note removed: "Add footprint for: Q1 D1,2"
- note removed: "Add value for: Q1 D1,2 R7, 8 L1"
- note removed: "Copy These passives when placing, they have 0603 and 0402 footprints respectively"
- note removed: "Do we want the features to be controlled via ESP?"
- note removed: "PLACE IF Vb =/= 4.05"
- moved on the sheet: C10, C11, C12, C13, C14, C15, C16, C17, C18, C19, C20, C21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

Commit message: Updated Schematic
added mounting holes, finished revision one, and unplaced/routed board (undone)
Parts:
- removed R17, R18, R19: 0, Resistor_SMD:R_0402_1005Metric, symbol Device:R_Small
- added H1, H2, H3, H4: MountingHole, MountingHole:MountingHole_2.2mm_M2_DIN965_Pad_TopBottom, symbol Mechanical:MountingHole
- C6: footprint Capacitor_SMD:C_0805_2012Metric -> Capacitor_SMD:C_0603_1608Metric
Connections:
- net demp is gone; now on net GND: U1.10 (DEMP)
- net flt is gone; now on net GND: U1.11 (FLT)
- net fmt is gone; now on net GND: U1.16 (FMT)
- net cap1: no longer C18.1, U1.2 (CAPP)
- net ts: now reaches R10.1, R9.2, U3.7 (TS)
- net test: now reaches R25.2, U2.7 (TEST2), U2.8 (TEST1)
- net mtdi: now reaches R14.2, U6.18 (MTDI)
- new net capp: C18.1, U1.2 (CAPP)
